Commit message: Added robotiq gripper support, added srdf for all rox drives, refactored launch files

File: neo_rox_moveit2/srdf/rox.srdf.xacro (robot description, xacro)
@@ -5,148 +5,95 @@
 -->
 <robot xmlns:xacro="http://www.ros.org/wiki/xacro" name="rox">
-     <xacro:arg name="prefix" default=""/>
-     <xacro:property name="prefix_value" value="$(arg prefix)"/>
-    <!--GROUPS: Representation of a set of joints and links. This can be useful for specifying DOF to plan for, defining arms, end effectors, etc-->
-    <!--LINKS: When a link is specified, the parent joint of that link (if it exists) is automatically included-->
-    <!--JOINTS: When a joint is specified, the child link of that joint (which will always exist) is automatically included-->
-    <!--CHAINS: When a chain is specified, all the links along the chain (including endpoints) are included in the group. Additionally, all the joints that are parents to included links are also included. This means that joints along the chain and the parent joint of the base link are included in the group-->
-    <!--SUBGROUPS: Groups can also be formed by referencing to already defined group names-->
-    <group name="ur_manipulator">
-        <joint name="${prefix_value}wrist_1_joint"/>
-        <joint name="${prefix_value}wrist_2_joint"/>
-        <joint name="${prefix_value}wrist_3_joint"/>
-        <joint name="${prefix_value}shoulder_pan_joint"/>
-        <joint name="${prefix_value}shoulder_lift_joint"/>
-        <joint name="${prefix_value}elbow_joint"/>
-        <chain base_link="${prefix_value}base_link" tip_link="${prefix_value}tool0"/>
-    </group>
-    <!--GROUP STATES: Purpose: Define a named state for a particular group, in terms of joint values. This is useful to define states like 'folded arms'-->
-    <group_state name="up" group="ur_manipulator">
-      <joint name="${prefix_value}elbow_joint" value="0" />
-      <joint name="${prefix_value}shoulder_lift_joint" value="-1.5707" />
-      <joint name="${prefix_value}shoulder_pan_joint" value="0" />
-      <joint name="${prefix_value}wrist_1_joint" value="-1.5707" />
-      <joint name="${prefix_value}wrist_2_joint" value="0" />
-      <joint name="${prefix_value}wrist_3_joint" value="0" />
-    </group_state>
-    <group_state name="test_configuration" group="ur_manipulator">
-      <joint name="${prefix_value}elbow_joint" value="1.83" />
-      <joint name="${prefix_value}shoulder_lift_joint" value="-2.66" />
-      <joint name="${prefix_value}shoulder_pan_joint" value="3.14" />
-      <joint name="${prefix_value}wrist_1_joint" value="-1.45" />
-      <joint name="${prefix_value}wrist_2_joint" value="3.22" />
-      <joint name="${prefix_value}wrist_3_joint" value="4.75" />
-    </group_state>
-    <!--DISABLE COLLISIONS: By default it is assumed that any link of the robot could potentially come into collision with any other link in the robot. This tag disables collision checking between a specified pair of links. -->
-    <disable_collisions link1="base_footprint" link2="cabinet_link" reason="Adjacent"/>
-    <disable_collisions link1="base_footprint" link2="lidar_1_link" reason="Adjacent"/>
-    <disable_collisions link1="base_footprint" link2="lidar_2_link" reason="Adjacent"/>
-    <disable_collisions link1="base_footprint" link2="caster_back_left_link" reason="Adjacent"/>
-    <disable_collisions link1="base_footprint" link2="caster_back_right_link" reason="Adjacent"/>
-    <disable_collisions link1="base_footprint" link2="caster_front_left_link" reason="Adjacent"/>
-    <disable_collisions link1="base_footprint" link2="caster_front_right_link" reason="Adjacent"/>
-    <disable_collisions link1="base_footprint" link2="wheel_back_left_link" reason="Never"/>
-    <disable_collisions link1="base_footprint" link2="wheel_back_right_link" reason="Never"/>
-    <disable_collisions link1="base_footprint" link2="wheel_front_left_link" reason="Never"/>
-    <disable_collisions link1="base_footprint" link2="wheel_front_right_link" reason="Never"/>
-    <disable_collisions link1="base_footprint" link2="${prefix_value}base_link_inertia" reason="Never"/>
-    <disable_collisions link1="base_footprint" link2="${prefix_value}shoulder_link" reason="Never"/>
-    <disable_collisions link1="cabinet_link" link2="lidar_1_link" reason="Adjacent"/>
-    <disable_collisions link1="cabinet_link" link2="lidar_2_link" reason="Adjacent"/>
-    <disable_collisions link1="cabinet_link" link2="caster_back_left_link" reason="Never"/>
-    <disable_collisions link1="cabinet_link" link2="caster_back_right_link" reason="Never"/>
-    <disable_collisions link1="cabinet_link" link2="caster_front_left_link" reason="Never"/>
-    <disable_collisions link1="cabinet_link" link2="caster_front_right_link" reason="Never"/>
-    <disable_collisions link1="cabinet_link" link2="wheel_back_left_link" reason="Never"/>
-    <disable_collisions link1="cabinet_link" link2="wheel_back_right_link" reason="Never"/>
-    <disable_collisions link1="cabinet_link" link2="wheel_front_left_link" reason="Never"/>
-    <disable_collisions link1="cabinet_link" link2="wheel_front_right_link" reason="Never"/>
-    <disable_collisions link1="cabinet_link" link2="${prefix_value}base_link_inertia" reason="Adjacent"/>
-    <disable_collisions link1="cabinet_link" link2="${prefix_value}shoulder_link" reason="Never"/>
-    <disable_collisions link1="lidar_1_link" link2="lidar_2_link" reason="Adjacent"/>
-    <disable_collisions link1="lidar_1_link" link2="caster_back_left_link" reason="Never"/>
-    <disable_collisions link1="lidar_1_link" link2="caster_back_right_link" reason="Never"/>
-    <disable_collisions link1="lidar_1_link" link2="caster_front_left_link" reason="Never"/>
-    <disable_collisions link1="lidar_1_link" link2="caster_front_right_link" reason="Never"/>
-    <disable_collisions link1="lidar_1_link" link2="wheel_back_left_link" reason="Never"/>
-    <disable_collisions link1="lidar_1_link" link2="wheel_back_right_link" reason="Never"/>
-    <disable_collisions link1="lidar_1_link" link2="wheel_front_left_link" reason="Never"/>
-    <disable_collisions link1="lidar_1_link" link2="wheel_front_right_link" reason="Never"/>
-    <disable_collisions link1="lidar_1_link" link2="${prefix_value}base_link_inertia" reason="Never"/>
-    <disable_collisions link1="lidar_1_link" link2="${prefix_value}shoulder_link" reason="Never"/>
-    <disable_collisions link1="lidar_2_link" link2="caster_back_left_link" reason="Never"/>
-    <disable_collisions link1="lidar_2_link" link2="caster_back_right_link" reason="Never"/>
-    <disable_collisions link1="lidar_2_link" link2="caster_front_left_link" reason="Never"/>
-    <disable_collisions link1="lidar_2_link" link2="caster_front_right_link" reason="Never"/>
-    <disable_collisions link1="lidar_2_link" link2="wheel_back_left_link" reason="Never"/>
-    <disable_collisions link1="lidar_2_link" link2="wheel_back_right_link" reason="Never"/>
-    <disable_collisions link1="lidar_2_link" link2="wheel_front_left_link" reason="Never"/>
-    <disable_collisions link1="lidar_2_link" link2="wheel_front_right_link" reason="Never"/>
-    <disable_collisions link1="lidar_2_link" link2="${prefix_value}base_link_inertia" reason="Never"/>
-    <disable_collisions link1="lidar_2_link" link2="${prefix_value}shoulder_link" reason="Never"/>
-    <disable_collisions link1="lidar_2_link" link2="${prefix_value}upper_arm_link" reason="Never"/>
-    <disable_collisions link1="caster_back_left_link" link2="caster_back_right_link" reason="Never"/>
-    <disable_collisions link1="caster_back_left_link" link2="caster_front_left_link" reason="Never"/>
-    <disable_collisions link1="caster_back_left_link" link2="caster_front_right_link" reason="Never"/>
-    <disable_collisions link1="caster_back_left_link" link2="wheel_back_left_link" reason="Adjacent"/>
-    <disable_collisions link1="caster_back_left_link" link2="wheel_back_right_link" reason="Never"/>
-    <disable_collisions link1="caster_back_left_link" link2="wheel_front_left_link" reason="Never"/>
-    <disable_collisions link1="caster_back_left_link" link2="wheel_front_right_link" reason="Never"/>
-    <disable_collisions link1="caster_back_left_link" link2="${prefix_value}base_link_inertia" reason="Never"/>
-    <disable_collisions link1="caster_back_left_link" link2="${prefix_value}shoulder_link" reason="Never"/>
-    <disable_collisions link1="caster_back_left_link" link2="${prefix_value}upper_arm_link" reason="Never"/>
-    <disable_collisions link1="caster_back_right_link" link2="caster_front_left_link" reason="Never"/>
-    <disable_collisions link1="caster_back_right_link" link2="caster_front_right_link" reason="Never"/>
-    <disable_collisions link1="caster_back_right_link" link2="wheel_back_left_link" reason="Never"/>
-    <disable_collisions link1="caster_back_right_link" link2="wheel_back_right_link" reason="Adjacent"/>
-    <disable_collisions link1="caster_back_right_link" link2="wheel_front_left_link" reason="Never"/>
-    <disable_collisions link1="caster_back_right_link" link2="wheel_front_right_link" reason="Never"/>
-    <disable_collisions link1="caster_back_right_link" link2="${prefix_value}base_link_inertia" reason="Never"/>
-    <disable_collisions link1="caster_back_right_link" link2="${prefix_value}shoulder_link" reason="Never"/>
-    <disable_collisions link1="caster_back_right_link" link2="${prefix_value}upper_arm_link" reason="Never"/>
-    <disable_collisions link1="caster_front_left_link" link2="caster_front_right_link" reason="Never"/>
-    <disable_collisions link1="caster_front_left_link" link2="wheel_back_left_link" reason="Never"/>
-    <disable_collisions link1="caster_front_left_link" link2="wheel_back_right_link" reason="Never"/>
-    <disable_collisions link1="caster_front_left_link" link2="wheel_front_left_link" reason="Adjacent"/>
-    <disable_collisions link1="caster_front_left_link" link2="wheel_front_right_link" reason="Never"/>
-    <disable_collisions link1="caster_front_left_link" link2="${prefix_value}base_link_inertia" reason="Never"/>
-    <disable_collisions link1="caster_front_left_link" link2="${prefix_value}shoulder_link" reason="Never"/>
-    <disable_collisions link1="caster_front_right_link" link2="wheel_back_left_link" reason="Never"/>
-    <disable_collisions link1="caster_front_right_link" link2="wheel_back_right_link" reason="Never"/>
-    <disable_collisions link1="caster_front_right_link" link2="wheel_front_left_link" reason="Never"/>
-    <disable_collisions link1="caster_front_right_link" link2="wheel_front_right_link" reason="Adjacent"/>
-    <disable_collisions link1="caster_front_right_link" link2="${prefix_value}base_link_inertia" reason="Never"/>
-    <disable_collisions link1="caster_front_right_link" link2="${prefix_value}shoulder_link" reason="Never"/>
-    <disable_collisions link1="wheel_back_left_link" link2="wheel_back_right_link" reason="Never"/>
-    <disable_collisions link1="wheel_back_left_link" link2="wheel_front_left_link" reason="Never"/>
-    <disable_collisions link1="wheel_back_left_link" link2="wheel_front_right_link" reason="Never"/>
-    <disable_collisions link1="wheel_back_left_link" link2="${prefix_value}base_link_inertia" reason="Never"/>
-    <disable_collisions link1="wheel_back_left_link" link2="${prefix_value}shoulder_link" reason="Never"/>
-    <disable_collisions link1="wheel_back_left_link" link2="${prefix_value}upper_arm_link" reason="Never"/>
-    <disable_collisions link1="wheel_back_right_link" link2="wheel_front_left_link" reason="Never"/>
-    <disable_collisions link1="wheel_back_right_link" link2="wheel_front_right_link" reason="Never"/>
-    <disable_collisions link1="wheel_back_right_link" link2="${prefix_value}base_link_inertia" reason="Never"/>
-    <disable_collisions link1="wheel_back_right_link" link2="${prefix_value}shoulder_link" reason="Never"/>
-    <disable_collisions link1="wheel_back_right_link" link2="${prefix_value}upper_arm_link" reason="Never"/>
-    <disable_collisions link1="wheel_front_left_link" link2="wheel_front_right_link" reason="Never"/>
-    <disable_collisions link1="wheel_front_left_link" link2="${prefix_value}base_link_inertia" reason="Never"/>
-    <disable_collisions link1="wheel_front_left_link" link2="${prefix_value}shoulder_link" reason="Never"/>
-    <disable_collisions link1="wheel_front_left_link" link2="${prefix_value}upper_arm_link" reason="Never"/>
-    <disable_collisions link1="wheel_front_right_link" link2="${prefix_value}base_link_inertia" reason="Never"/>
-    <disable_collisions link1="wheel_front_right_link" link2="${prefix_value}shoulder_link" reason="Never"/>
-    <disable_collisions link1="wheel_front_right_link" link2="${prefix_value}upper_arm_link" reason="Never"/>
-    <disable_collisions link1="${prefix_value}base_link_inertia" link2="${prefix_value}shoulder_link" reason="Adjacent"/>
-    <disable_collisions link1="${prefix_value}base_link_inertia" link2="${prefix_value}upper_arm_link" reason="Never"/>
-    <disable_collisions link1="${prefix_value}base_link_inertia" link2="${prefix_value}wrist_1_link" reason="Never"/>
-    <disable_collisions link1="${prefix_value}forearm_link" link2="${prefix_value}upper_arm_link" reason="Adjacent"/>
-    <disable_collisions link1="${prefix_value}forearm_link" link2="${prefix_value}wrist_1_link" reason="Adjacent"/>
-    <disable_collisions link1="${prefix_value}shoulder_link" link2="${prefix_value}upper_arm_link" reason="Adjacent"/>
-    <disable_collisions link1="${prefix_value}shoulder_link" link2="${prefix_value}wrist_1_link" reason="Never"/>
-    <disable_collisions link1="${prefix_value}shoulder_link" link2="${prefix_value}wrist_2_link" reason="Never"/>
-    <disable_collisions link1="${prefix_value}wrist_1_link" link2="${prefix_value}wrist_2_link" reason="Adjacent"/>
-    <disable_collisions link1="${prefix_value}wrist_1_link" link2="${prefix_value}wrist_3_link" reason="Never"/>
-    <disable_collisions link1="${prefix_value}wrist_2_link" link2="${prefix_value}wrist_3_link" reason="Adjacent"/>
-    <disable_collisions link1="${prefix_value}tool0" link2="${prefix_value}wrist_1_link" reason="Never" />
-    <disable_collisions link1="${prefix_value}tool0" link2="${prefix_value}wrist_2_link" reason="Never" />
-    <disable_collisions link1="${prefix_value}tool0" link2="${prefix_value}wrist_3_link" reason="Adjacent" />
+  <xacro:arg name="prefix" default=""/>
+  <xacro:arg name="rox_type" default="argo"/>
+  <xacro:arg name="gripper_type" default=""/>
+  <xacro:property name="prefix_value" value="$(arg prefix)"/>
+  <xacro:property name="rox_typ" value="$(arg rox_type)"/>
+  <xacro:property name="gripper" value="$(arg gripper_type)"/>
+  <!--GROUPS: Representation of a set of joints and links. This can be useful for specifying DOF to plan for, defining arms, end effectors, etc-->
+  <!--LINKS: When a link is specified, the parent joint of that link (if it exists) is automatically included-->
+  <!--JOINTS: When a joint is specified, the child link of that joint (which will always exist) is automatically included-->
+  <!--CHAINS: When a chain is specified, all the links along the chain (including endpoints) are included in the group. Additionally, all the joints that are parents to included links are also included. This means that joints along the chain and the parent joint of the base link are included in the group-->
+  <!--SUBGROUPS: Groups can also be formed by referencing to already defined group names-->
+  <group name="ur_manipulator">
+      <joint name="${prefix_value}wrist_1_joint"/>
+      <joint name="${prefix_value}wrist_2_joint"/>
+      <joint name="${prefix_value}wrist_3_joint"/>
+      <joint name="${prefix_value}shoulder_pan_joint"/>
+      <joint name="${prefix_value}shoulder_lift_joint"/>
+      <joint name="${prefix_value}elbow_joint"/>
+      <chain base_link="${prefix_value}base_link" tip_link="${prefix_value}tool0"/>
+  </group>
+  <!--GROUP STATES: Purpose: Define a named state for a particular group, in terms of joint values. This is useful to define states like 'folded arms'-->
+  <group_state name="up" group="ur_manipulator">
+    <joint name="${prefix_value}elbow_joint" value="0" />
+    <joint name="${prefix_value}shoulder_lift_joint" value="-1.5707" />
+    <joint name="${prefix_value}shoulder_pan_joint" value="0" />
+    <joint name="${prefix_value}wrist_1_joint" value="-1.5707" />
+    <joint name="${prefix_value}wrist_2_joint" value="0" />
+    <joint name="${prefix_value}wrist_3_joint" value="0" />
+  </group_state>
+  <group_state name="test_configuration" group="ur_manipulator">
+    <joint name="${prefix_value}elbow_joint" value="1.83" />
+    <joint name="${prefix_value}shoulder_lift_joint" value="-2.66" />
+    <joint name="${prefix_value}shoulder_pan_joint" value="3.14" />
+    <joint name="${prefix_value}wrist_1_joint" value="-1.45" />
+    <joint name="${prefix_value}wrist_2_joint" value="3.22" />
+    <joint name="${prefix_value}wrist_3_joint" value="4.75" />
+  </group_state>
+  <!--DISABLE COLLISIONS: By default it is assumed that any link of the robot could potentially come into collision with any other link in the robot. This tag disables collision checking between a specified pair of links. -->
+  <!-- Common collisions for all rox drives-->
+  <disable_collisions link1="base_footprint" link2="cabinet_link" reason="Adjacent"/>
+  <disable_collisions link1="base_footprint" link2="lidar_1_link" reason="Adjacent"/>
+  <disable_collisions link1="base_footprint" link2="lidar_2_link" reason="Adjacent"/>
+  <disable_collisions link1="base_footprint" link2="${prefix_value}base_link_inertia" reason="Never"/>
+  <disable_collisions link1="base_footprint" link2="${prefix_value}shoulder_link" reason="Never"/>
+  <disable_collisions link1="lidar_1_link" link2="${prefix_value}base_link_inertia" reason="Never"/>
+  <disable_collisions link1="lidar_1_link" link2="${prefix_value}shoulder_link" reason="Never"/>
+  <disable_collisions link1="lidar_1_link" link2="lidar_2_link" reason="Adjacent"/>
+  <disable_collisions link1="lidar_2_link" link2="${prefix_value}base_link_inertia" reason="Never"/>
+  <disable_collisions link1="lidar_2_link" link2="${prefix_value}shoulder_link" reason="Never"/>
+  <disable_collisions link1="lidar_2_link" link2="${prefix_value}upper_arm_link" reason="Never"/>
+  <disable_collisions link1="cabinet_link" link2="lidar_1_link" reason="Adjacent"/>
+  <disable_collisions link1="cabinet_link" link2="lidar_2_link" reason="Adjacent"/>
+  <disable_collisions link1="cabinet_link" link2="${prefix_value}base_link_inertia" reason="Adjacent"/>
+  <disable_collisions link1="cabinet_link" link2="${prefix_value}shoulder_link" reason="Never"/>
+  <disable_collisions link1="${prefix_value}base_link_inertia" link2="${prefix_value}shoulder_link" reason="Adjacent"/>
+  <disable_collisions link1="${prefix_value}base_link_inertia" link2="${prefix_value}upper_arm_link" reason="Never"/>
+  <disable_collisions link1="${prefix_value}base_link_inertia" link2="${prefix_value}wrist_1_link" reason="Never"/>
+  <disable_collisions link1="${prefix_value}base_link_inertia" link2="${prefix_value}wrist_2_link" reason="Never"/>
+  <disable_collisions link1="${prefix_value}forearm_link" link2="${prefix_value}upper_arm_link" reason="Adjacent"/>
+  <disable_collisions link1="${prefix_value}forearm_link" link2="${prefix_value}wrist_1_link" reason="Adjacent"/>
+  <disable_collisions link1="${prefix_value}shoulder_link" link2="${prefix_value}upper_arm_link" reason="Adjacent"/>
+  <disable_collisions link1="${prefix_value}shoulder_link" link2="${prefix_value}wrist_1_link" reason="Never"/>
+  <disable_collisions link1="${prefix_value}shoulder_link" link2="${prefix_value}wrist_2_link" reason="Never"/>
+  <disable_collisions link1="${prefix_value}wrist_1_link" link2="${prefix_value}wrist_2_link" reason="Adjacent"/>
+  <disable_collisions link1="${prefix_value}wrist_1_link" link2="${prefix_value}wrist_3_link" reason="Never"/>
+  <disable_collisions link1="${prefix_value}wrist_2_link" link2="${prefix_value}wrist_3_link" reason="Adjacent"/>
+  <disable_collisions link1="${prefix_value}tool0" link2="${prefix_value}wrist_1_link" reason="Never" />
+  <disable_collisions link1="${prefix_value}tool0" link2="${prefix_value}wrist_2_link" reason="Never" />
+  <disable_collisions link1="${prefix_value}tool0" link2="${prefix_value}wrist_3_link" reason="Adjacent" />
+  <xacro:if value="${rox_typ == 'argo' or rox_typ == 'argo-trio'}">
+    <xacro:include filename="$(find neo_rox_moveit2)/srdf/rox_argo.srdf.xacro" />
+    <xacro:rox_argo/>
+  </xacro:if>
+  <xacro:if value="${rox_typ == 'diff' or rox_typ == 'trike'}">
+    <xacro:include filename="$(find neo_rox_moveit2)/srdf/rox_diff.srdf.xacro" />
+    <xacro:rox_diff/>
+  </xacro:if>
+  <!-- Gripper Conditions -->
+  <xacro:unless value="${gripper == ''}">
+    <xacro:if value="${gripper == '2f_140'}">
+      <xacro:include filename="$(find neo_rox_moveit2)/srdf/robotiq_2f_140.srdf.xacro" />
+      <xacro:robotiq_2f_140 />
+    </xacro:if>
+    <xacro:if value="${gripper == '2f_85'}">
+      <xacro:include filename="$(find neo_rox_moveit2)/srdf/robotiq_2f_85.srdf.xacro" />
+      <xacro:robotiq_2f_85 />
+    </xacro:if>
+    <xacro:if value="${gripper == 'epick'}">
+      <xacro:include filename="$(find neo_rox_moveit2)/srdf/robotiq_epick.xacro" />
+      <xacro:robotiq_epick />
+    </xacro:if>
+  </xacro:unless>
 </robot>
